File: hardware/dasblinkenhat-controller-mk-2.0.brd (EAGLE design)
At the start: 57.1 x 12.7 mm, 12 parts, among them IC1 TINY85, J1 M03JST-XH-RA-PTH

Commit message: minor silk tweak
Parts:
- removed U$1: (no value), a_parts:CC-BY-SA-4.0-NO-URL
Routing:
- net VCC: track 0.00 -> 70.6 mm
- net BUTT: track 0.00 -> 29.4 mm
- net SPEED: track 0.00 -> 20.4 mm
- net DAT: track 0.00 -> 18.6 mm
- net BRIGHT: track 0.00 -> 13.5 mm
- net RST: track 0.00 -> 2.80 mm
Changed lines of the file:
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@@
 <attribute name="NAME" x="8.89" y="11.049" size="0.8" layer="25" font="vector" ratio="12" align="bottom-center"/>
 </element>
-<element name="U$1" library="a_parts" package="CC-BY-SA-4.0-NO-URL" value="" x="18.415" y="6.35" rot="MR0"/>
 <element name="U$2" library="a_parts" package="OSHWLOGO_TINY_SILKONLY" value="" x="10.16" y="1.905" rot="MR0"/>
 </elements>
@@
 <contactref element="R3" pad="1"/>
 <contactref element="R2" pad="1"/>
-<wire x1="40.64" y1="6.35" x2="54.39" y2="4.445" width="0" layer="19" extent="1-1"/>
-<wire x1="31.75" y1="6.35" x2="40.64" y2="6.35" width="0" layer="19" extent="1-1"/>
-<wire x1="15.24" y1="10.16" x2="31.75" y2="6.35" width="0" layer="19" extent="1-1"/>
-<wire x1="12.7" y1="10.16" x2="15.24" y2="10.16" width="0" layer="19" extent="1-1"/>
-<wire x1="8.89" y1="9.255" x2="12.7" y2="10.16" width="0" layer="19" extent="1-1"/>
-<wire x1="5.08" y1="8.85" x2="8.89" y2="9.255" width="0" layer="19" extent="1-1"/>
-<wire x1="7.62" y1="3.175" x2="8.89" y2="9.255" width="0" layer="19" extent="1-1"/>
+<wire x1="54.39" y1="4.445" x2="54.39" y2="6.57" width="1" layer="16"/>
+<wire x1="54.39" y1="6.57" x2="53.34" y2="7.62" width="1" layer="16"/>
+<wire x1="53.34" y1="7.62" x2="42.545" y2="7.62" width="1" layer="16"/>
+<wire x1="42.545" y1="7.62" x2="41.91" y2="8.255" width="1" layer="16"/>
+<wire x1="41.91" y1="8.255" x2="33.655" y2="8.255" width="1" layer="16"/>
+<wire x1="33.655" y1="8.255" x2="14.605" y2="8.255" width="1" layer="16"/>
+<wire x1="14.605" y1="8.255" x2="12.7" y2="10.16" width="1" layer="16"/>
+<wire x1="12.7" y1="10.16" x2="9.795" y2="10.16" width="1" layer="16"/>
+<wire x1="9.795" y1="10.16" x2="8.89" y2="9.255" width="1" layer="16"/>
+<wire x1="8.89" y1="9.255" x2="5.485" y2="9.255" width="1" layer="16"/>
+<wire x1="5.485" y1="9.255" x2="5.08" y2="8.85" width="1" layer="16"/>
+<wire x1="15.24" y1="10.16" x2="12.7" y2="10.16" width="0.635" layer="16"/>
+<wire x1="7.62" y1="3.175" x2="8.255" y2="3.175" width="0.4064" layer="16"/>
+<wire x1="8.255" y1="3.175" x2="10.795" y2="5.715" width="0.4064" layer="16"/>
+<wire x1="10.795" y1="5.715" x2="10.795" y2="8.255" width="0.4064" layer="16"/>
+<wire x1="10.795" y1="8.255" x2="12.7" y2="10.16" width="0.4064" layer="16"/>
+<wire x1="42.545" y1="7.62" x2="41.91" y2="7.62" width="0.4064" layer="16"/>
+<wire x1="41.91" y1="7.62" x2="40.64" y2="6.35" width="0.4064" layer="16"/>
+<wire x1="31.75" y1="6.35" x2="33.655" y2="8.255" width="0.4064" layer="16"/>
 </signal>
 <signal name="RST">
 <contactref element="IC1" pad="1"/>
 <contactref element="R1" pad="P$1"/>
-<wire x1="12.7" y1="3.175" x2="15.24" y2="2.54" width="0" layer="19" extent="1-1"/>
+<wire x1="12.7" y1="3.175" x2="14.605" y2="3.175" width="0.4064" layer="1"/>
+<wire x1="14.605" y1="3.175" x2="15.24" y2="2.54" width="0.4064" layer="1"/>
 </signal>
 <signal name="DAT">
 <contactref element="J1" pad="2"/>
 <contactref element="IC1" pad="6"/>
-<wire x1="5.08" y1="6.35" x2="20.32" y2="10.16" width="0" layer="19" extent="1-1"/>
+<wire x1="5.08" y1="6.35" x2="6.35" y2="5.08" width="0.4064" layer="1"/>
+<wire x1="6.35" y1="5.08" x2="16.51" y2="5.08" width="0.4064" layer="1"/>
+<wire x1="16.51" y1="5.08" x2="20.32" y2="8.89" width="0.4064" layer="1"/>
+<wire x1="20.32" y1="8.89" x2="20.32" y2="10.16" width="0.4064" layer="1"/>
 </signal>
 <signal name="BUTT">
@@
 <contactref element="BUTT" pad="2"/>
 <contactref element="IC1" pad="5"/>
-<wire x1="44.105" y1="3.1" x2="44.105" y2="9.6" width="0" layer="19" extent="1-1"/>
-<wire x1="22.86" y1="10.16" x2="44.105" y2="9.6" width="0" layer="19" extent="1-1"/>
+<wire x1="22.86" y1="10.16" x2="24.13" y2="8.89" width="0.4064" layer="1"/>
+<wire x1="24.13" y1="8.89" x2="41.275" y2="8.89" width="0.4064" layer="1"/>
+<wire x1="41.275" y1="8.89" x2="44.105" y2="6.06" width="0.4064" layer="1"/>
+<wire x1="44.105" y1="6.06" x2="44.105" y2="3.1" width="0.4064" layer="1"/>
+<wire x1="44.105" y1="9.6" x2="44.105" y2="6.06" width="0.4064" layer="1"/>
 </signal>
 <signal name="SPEED">
 <contactref element="R3" pad="2"/>
 <contactref element="IC1" pad="3"/>
-<wire x1="20.32" y1="2.54" x2="38.1" y2="3.81" width="0" layer="19" extent="1-1"/>
+<wire x1="20.32" y1="2.54" x2="22.225" y2="4.445" width="0.4064" layer="1"/>
+<wire x1="22.225" y1="4.445" x2="24.13" y2="4.445" width="0.4064" layer="1"/>
+<wire x1="24.13" y1="4.445" x2="26.67" y2="1.905" width="0.4064" layer="1"/>
+<wire x1="26.67" y1="1.905" x2="36.195" y2="1.905" width="0.4064" layer="1"/>
+<wire x1="36.195" y1="1.905" x2="38.1" y2="3.81" width="0.4064" layer="1"/>
 </signal>
 <signal name="BRIGHT">
 <contactref element="R2" pad="2"/>
 <contactref element="IC1" pad="2"/>
-<wire x1="17.78" y1="2.54" x2="29.21" y2="3.81" width="0" layer="19" extent="1-1"/>
+<wire x1="17.78" y1="2.54" x2="20.955" y2="5.715" width="0.4064" layer="1"/>
+<wire x1="20.955" y1="5.715" x2="24.765" y2="5.715" width="0.4064" layer="1"/>
+<wire x1="24.765" y1="5.715" x2="26.67" y2="3.81" width="0.4064" layer="1"/>
+<wire x1="26.67" y1="3.81" x2="29.21" y2="3.81" width="0.4064" layer="1"/>
 </signal>
 </signals>
