File: hardware/dasblinkenhat-controller-mk-4.0.brd (EAGLE design)
At the start: 50.8 x 22.9 mm, 13 parts, among them J1 M03JST-XH-RA-PTH, U1 ADAFRUIT_FEATHER_SHIELD

Commit message: new hardware rev off to fab
Parts:
- removed BAT: M02JST-2MM-SMT, a_parts:JST-2-SMD
- removed BUTT: DTS-6MM, A_butts:DTSM-6
- removed F1: 2A, a_parts:PTC-1206
- removed PWR: (no value), a_parts:PUSHBUTTON-CW-SPST-12MM
- removed R1: 27R, a_parts:R0805
- removed R2: 100R, a_parts:R0805
- removed TP1: BRIGHT, a_parts:EVM3Y
- added BATT: M02JST-2MM-SMT, a_parts:JST-2-SMD
- added BRIGHT, DELAY: 10K, a_parts:EVM3Y
- added D1: MBRA140, a_parts:SMA-DIODE-SCHOTTKY
- added IC1: SN74LVC1T45, a_parts:SOT23-6
- added MODE: DTS-6MM, A_butts:DTSM-6
- added POWER: PUSHBUTTON-LATCHING-SPST12MM-PTH, a_parts:PUSHBUTTON-CW-SPST-12MM
- added SKIP_LVC: JUMPER-PAD-2-NOYES_SILK, a_parts:PAD-JUMPER-2-NO_YES_SILK
- moved U$2 60.2 mm to (7.62, 3.81)
- moved J1 1.27 mm to (43.2, 11.4)
- flipped C1 to the top
- flipped C2 to the top
Connections:
- removed net BUTT: BUTT.1, BUTT.2, U1.9
- removed net DAT: R1.1, U1.6
- removed net N$2: F1.1, PWR.2
- removed net N$3: J1.2, R1.2
- removed net N$4: R2.1, TP1.E
- new net BATT_DIV: U1.9
- new net DATA_IN: IC1.4, SKIP_LVC.1, U1.5
- new net DATA_OUT: IC1.3, J1.2, SKIP_LVC.2
- new net MODE: MODE.1, MODE.2, U1.6
- new net SPEED: DELAY.S, U1.A3
- new net VUSB: D1.A, U1.USB
- net BRIGHT: now also BRIGHT.S; no longer TP1.S
- net GND: now also BATT.1, BRIGHT.A, DELAY.A, IC1.2, IC1.5, MODE.3, MODE.4; no longer BAT.1, BUTT.3, BUTT.4, TP1.A
- net N$1: now also BATT.2, POWER.2; no longer BAT.2, PWR.1
- net VBATT+: now also D1.C, IC1.1, POWER.1; no longer F1.2
- net VCC: now also BRIGHT.E, DELAY.E, IC1.6; no longer R2.2
Routing:
- net VBATT+: track 0.00 -> 64.8 mm, vias 0 -> 2
- net VCC: track 0.00 -> 36.7 mm, vias 0 -> 2
- net MODE: track 0.00 -> 28.5 mm
- net DATA_OUT: track 0.00 -> 15.4 mm
- net BRIGHT: track 0.00 -> 11.6 mm
- net DATA_IN: track 0.00 -> 10.8 mm
- net N$1: track 0.00 -> 10.7 mm
- net VUSB: track 0.00 -> 6.29 mm
- net SPEED: track 0.00 -> 5.45 mm
Other:
- outline, holes or cut-outs redrawn
