File: hardware/dasblinkenhat-controller-mk-4.0.sch (EAGLE design)
At the start: 12 parts, among them J1 M03JST-XH-RA-PTH, U1 ADAFRUIT_FEATHER_SHIELD

Commit message: new hardware rev off to fab
Parts:
- removed BAT: M02JST-2MM-SMT, a_parts:M02JST-2MM-SMT
- removed F1: 2A, a_parts:PTCSMD
- removed PWR: PUSHBUTTON-LATCHING-SPST12MM-PTH, a_parts:PUSHBUTTON-LATCHING-SPST12MM-PTH
- removed R1: 27R, a_parts:RESISTORR0805
- removed R2: 100R, a_parts:RESISTORR0805
- removed TP1: BRIGHT, a_parts:POTENTIOMETEREVM3Y
- added BATT: M02JST-2MM-SMT, a_parts:M02JST-2MM-SMT
- added BRIGHT, DELAY: 10K, a_parts:POTENTIOMETEREVM3Y
- added D1: MBRA140, a_parts:DIODE-SCHOTTKYSMA
- added IC1: SN74LVC1T45, a_parts:SN74LVC1T45SOT23-6
- added POWER: PUSHBUTTON-LATCHING-SPST12MM-PTH, a_parts:PUSHBUTTON-LATCHING-SPST12MM-PTH
- added SKIP_LVC: JUMPER-PAD-2-NOYES_SILK, a_parts:JUMPER-PAD-2-NOYES_SILK
- renumbered BUTT to MODE
Connections:
- removed net BUTT: MODE.1, U1.9
- removed net DAT: R1.1, U1.6
- removed net N$2: F1.1, PWR.NC
- removed net N$3: J1.2, R1.2
- removed net N$4: R2.1, TP1.E
- new net BATT_DIV: U1.9
- new net DATA_IN: IC1.B, SKIP_LVC.1, U1.5
- new net DATA_OUT: IC1.A, J1.2, SKIP_LVC.2
- new net MODE: MODE.1, U1.6
- new net SPEED: DELAY.S, U1.A3
- new net VUSB: D1.A, U1.USB
- net BRIGHT: now also BRIGHT.S; no longer TP1.S
- net GND: now also BATT.2, BRIGHT.A, DELAY.A, IC1.DIR, IC1.GND; no longer BAT.2, TP1.A
- net N$1: now also BATT.1, POWER.NC; no longer BAT.1, PWR.COM
- net VBATT+: now also D1.C, IC1.VCC, POWER.COM; no longer F1.2
- net VCC: now also BRIGHT.E, DELAY.E, IC1.VDD; no longer R2.2
